File: 3458A Ref A9 Clone/3458A Ref A9 Clone.kicad_pcb (KiCad board)
At the start: 4 copper layers, 50 x 42.5 mm, 44 parts, among them J400 Molex KK 254, J401 Molex KK 254, Q1 MMBF4392, Q401 BD139, U401 ADR/LTZ1000(A), U402 LT1013

Commit message: Update to REV β
Parts:
- added C1: 10n, Capacitor_SMD:C_1206_3216Metric, F.Cu at (158.4, 113.5)
- added R5: 19k6, Resistor_SMD:R_0805_2012Metric, F.Cu at (136.9, 103.0)
- added R6: 22k, Resistor_SMD:R_0805_2012Metric, F.Cu at (143.4, 104.3)
- R413: footprint Resistor_SMD:R_0805_2012Metric -> Resistor_SMD:R_1206_3216Metric
- R419: value 1470 -> 1k6; footprint Resistor_SMD:R_0805_2012Metric -> Resistor_SMD:R_1206_3216Metric
- TP1, TP2, TP3, TP4, TP5, TP6: footprint TestPoint:TestPoint_Pad_D2.0mm -> KiCad:PinSocket_1x01_P2.54mm_Vertical
- U401: value ADR/LTZ1000(A) -> ADR1000
- moved R2 19.3 mm to (136.9, 106.8)
- moved C4 18.2 mm to (143.8, 124.5), turned to 0 degrees
- moved R415 17.7 mm to (136.9, 111.0)
- moved RN1 17.0 mm to (136.9, 127.1), turned to 0 degrees
- moved REF** 16.6 mm to (174.2, 114.0)
- moved REF** 14.4 mm to (153.2, 96.1)
- moved R419 10.5 mm to (141.4, 100.2)
- moved REF** 4.28 mm to (176.1, 105.8)
- moved R421 3.98 mm to (161.0, 97.0), turned to 90 degrees
- moved C5 3.89 mm to (136.9, 114.4)
- moved R414 3.25 mm to (136.9, 118.6)
- moved TP5 2.46 mm to (177.5, 100.2), turned to -90 degrees
- moved R417 2.17 mm to (158.4, 118.6)
- moved JP1 2.16 mm to (169.6, 111.3)
- moved R413 2.16 mm to (169.7, 104.4)
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- renumbered C5 to C4, C6 to C5
Connections:
- RN1 pad 10: Net-(RN1E-R5.2) -> J400 (1): Temp
- RN1 pad 11: J400 (1): Temp -> Net-(RN1C-R3.2)
- RN1 pad 12: Net-(RN1E-R5.2) -> J400 (1): Temp
- RN1 pad 13: Net-(RN1B-R2.2) -> unconnected-(RN1D-R4.2-Pad13)
- RN1 pad 14: J400 (1): Temp -> Net-(RN1C-R3.2)
- RN1 pad 15: Net-(RN1B-R2.2) -> J400 (1): Temp
- RN1 pad 2: Net-(RN1A-R1.1) -> J400 (2): REF GND
- RN1 pad 3: J400 (2): REF GND -> Net-(RN1A-R1.1)
- RN1 pad 4: Net-(RN1D-R4.1) -> J400 (2): REF GND
- RN1 pad 5: Net-(RN1D-R4.1) -> J400 (2): REF GND
- RN1 pad 6: J400 (2): REF GND -> Net-(RN1F-R6.1)
- RN1 pad 7: Net-(RN1G-R7.1) -> J400 (2): REF GND
- RN1 pad 8: Net-(RN1G-R7.1) -> Net-(RN1F-R6.1)
- TP3 pad 1: Net-(U402B--) -> ZD-
Routing:
- net J400 (2): REF GND: track 108.4 -> 158.9 mm, vias 16 -> 21
- net J400 (1): Temp: track 82.9 -> 66.0 mm
- net -15: track 10.1 -> 20.8 mm, vias 0 -> 9
- net +7V REF: track 51.0 -> 40.5 mm, vias 18 -> 12
- net Net-(JP1-A): track 22.0 -> 13.8 mm, vias 3 -> 0
- net +18: track 40.6 -> 33.3 mm
- net Net-(RN1C-R3.2): track 0.00 -> 6.75 mm
- net Net-(C1-Pad1): track 25.9 -> 32.4 mm
- net Net-(U402B--): track 11.6 -> 5.40 mm
- net Net-(U402B-+): track 62.0 -> 56.1 mm
- net Net-(RN1F-R6.1): track 0.00 -> 5.48 mm
- net Net-(RN1E-R5.2): track 5.37 -> 0.00 mm
- net Net-(RN1B-R2.2): track 5.37 -> 0.00 mm
- net Net-(RN1G-R7.1): track 3.89 -> 0.00 mm
- net Net-(RN1D-R4.1): track 3.89 -> 0.00 mm
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- added copper zone on B.Cu, net -15
- added copper zone on F.Cu, net -15
Other:
- board text added: "+18"
- board text added: "+18H"
- board text added: "-15"
- board text added: "5"
- board text added: "GNDF"
- board text added: "GNDH"
- board text added: "GNDS"
- board text added: "HTR"
- board text added: "REF"
- board text added: "REV β 03458-665X9"
- board text added: "Temp"
- board text removed: "REV α 03458-66509"

Commit message: Update to REV A
Parts:
- removed JP1: Jumper, Jumper:SolderJumper-2_P1.3mm_Bridged_Pad1.0x1.5mm
- removed R3: 20R, Resistor_SMD:R_2512_6332Metric
- moved REF** 16.1 mm to (163.7, 101.9)
- moved R413 6.98 mm to (169.7, 111.4), turned to 180 degrees
- moved R6 2.01 mm to (145.0, 103.1), turned to 90 degrees
- moved C4 1.02 mm to (143.7, 123.4)
- moved R421 0.59 mm to (161.0, 96.4)
- moved TP3 0.59 mm to (143.7, 115.4)
- moved TP4 0.59 mm to (143.7, 118.0)
- moved R420 0.51 mm to (163.7, 110.6)
- moved TP1 0.18 mm to (143.7, 128.9)
- moved TP2 0.18 mm to (143.7, 131.4)
Connections:
- C2 pad 1: Net-(JP1-A) -> +7V REF
- U401 pad 3: Net-(JP1-A) -> +7V REF
Routing:
- net +7V REF: track 40.5 -> 54.7 mm
- net Net-(JP1-A): track 13.8 -> 0.00 mm
- net J400 (1): Temp: track 66.0 -> 69.0 mm
- net Net-(C1-Pad1): track 32.4 -> 31.4 mm
- net Net-(D401-A): track 37.5 -> 38.5 mm
- net J400 (2): REF GND: track 158.9 -> 159.8 mm
- net Net-(Q401-E): track 73.0 -> 73.7 mm
- net ZD-: track 46.0 -> 45.4 mm
- net Net-(Q1-S): track 3.34 -> 2.74 mm
Other:
- board text added: "REV A 03458-665X9"
- board text removed: "REV β 03458-665X9"

Commit message: Release REV B
Parts:
- added R3: 1k, Resistor_SMD:R_0805_2012Metric, F.Cu at (164.1, 98.6)
- added R7: 1k, Resistor_SMD:R_0805_2012Metric, F.Cu at (147.6, 111.5)
- C1: value 10n -> 1n
- C2: value 100n -> 10n
- C411: value 22n -> 100n
- C5: value 100n -> 1n
- R1: value 10k -> 1k
- R2: value 680k -> 68k*
- R415: value 68k -> 15K*
- R419: value 1k6 -> 1k43
- R6: value 22k -> 11k8
- moved C414 16.5 mm to (143.4, 109.0)
- moved R4 10.8 mm to (147.6, 109.0), turned to 180 degrees
- moved C4 7.14 mm to (149.0, 118.6), turned to 90 degrees
- moved C3 6.17 mm to (153.2, 115.1), turned to 0 degrees
- moved TP3 5.60 mm to (144.1, 121.0), turned to 180 degrees
- moved R416 5.21 mm to (153.2, 120.1)
- moved C411 4.70 mm to (144.1, 113.0), turned to -90 degrees
- moved Q401 4.58 mm to (176.3, 94.6), turned to 180 degrees
- moved R1 4.40 mm to (148.7, 114.8), turned to 180 degrees
- moved REF** 3.79 mm to (166.6, 104.3)
- moved C1 3.05 mm to (158.4, 110.5)
- moved R417 0.87 mm to (158.4, 119.5)
- moved C412 0.76 mm to (161.2, 110.5)
- moved R420 0.76 mm to (163.7, 109.9)
- moved TP4 0.67 mm to (144.1, 118.5), turned to 180 degrees
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Connections:
- C411 pad 1: Net-(U402B-+) -> Net-(C411-Pad1)
- Q1 pad 3: +7V REF -> Net-(Q1-G)
- R2 pad 2: Net-(U402B-+) -> Net-(C411-Pad1)
- R415 pad 2: Net-(U402B-+) -> Net-(C411-Pad1)
- U401 pad 5: Net-(U402B-+) -> Net-(C411-Pad1)
- U402 pad 1: Net-(C1-Pad1) -> Net-(U402A-+)
- U402 pad 2: Net-(U402A--) -> J400 (2): REF GND
- U402 pad 3: Net-(U402A-+) -> Net-(U402B-+)
- U402 pad 4: J400 (2): REF GND -> Net-(U402B--)
- U402 pad 5: Net-(U402B-+) -> Net-(D400-A)
- U402 pad 6: Net-(U402B--) -> +18
- U402 pad 7: Net-(D400-A) -> Net-(C1-Pad1)
- U402 pad 8: +18 -> Net-(U402A--)
Routing:
- net Net-(U402B-+): track 56.1 -> 2.20 mm
- net Net-(C411-Pad1): track 0.00 -> 51.2 mm
- net Net-(C414-Pad1): track 48.3 -> 64.5 mm, vias 0 -> 6
- net J400 (1): Temp: track 69.0 -> 59.5 mm, vias 6 -> 3
- net Net-(U402A--): track 10.6 -> 19.2 mm
- net Net-(D400-A): track 10.1 -> 5.44 mm
- net Net-(C1-Pad1): track 31.4 -> 27.5 mm
- net Net-(Q1-G): track 0.00 -> 3.16 mm
- net J400 (2): REF GND: track 159.8 -> 157.5 mm, vias 21 -> 18
- net ZD-: track 45.4 -> 43.6 mm
- net J401 (3): GND Heater: track 18.4 -> 19.7 mm
- net +7V REF: track 54.7 -> 55.8 mm
- net Net-(U402B--): track 5.40 -> 4.40 mm
- net -15: track 20.8 -> 21.6 mm
- net Net-(U402A-+): track 2.77 -> 2.18 mm
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Other:
- board text added: "Michael D. 12/2024"
- board text added: "REV B 03458-665X9"
- board text removed: "Michael D. 11/2024"
- board text removed: "REV A 03458-665X9"
