File: 3458A Ref A9 Clone/3458A Ref A9 Clone.kicad_sch (KiCad schematic)
At the start: 37 parts, among them J400 Molex KK 254, J401 Molex KK 254, Q1 MMBF4392, Q401 BD139, U401 ADR/LTZ1000(A), U402 LT1013

Commit message: Update to REV β
Parts:
- added C1: 10n, Capacitor_SMD:C_1206_3216Metric, symbol Device:C_Small
- added R5: 19k6, Resistor_SMD:R_0805_2012Metric, symbol Device:R
- added R6: 22k, Resistor_SMD:R_0805_2012Metric, symbol Device:R
- R413: footprint Resistor_SMD:R_0805_2012Metric -> Resistor_SMD:R_1206_3216Metric
- R419: value 1470 -> 1k6; footprint Resistor_SMD:R_0805_2012Metric -> Resistor_SMD:R_1206_3216Metric; Type Metal film (Susumu RR1220P) -> Metal film 1/4W (Susumu RG3216P)
- TP1, TP2, TP3, TP4, TP5, TP6: footprint TestPoint:TestPoint_Pad_D2.0mm -> KiCad:PinSocket_1x01_P2.54mm_Vertical
- U401: value ADR/LTZ1000(A) -> ADR1000
- renumbered C5 to C4, C6 to C5
Connections:
- net -15: now also R5.2, R6.2
- net GNDA: now also RN1.2 (R2.1), RN1.4 (R4.1), RN1.5 (R5.1), RN1.7 (R7.1), R5.1, R6.1; no longer RN1.3 (R3.1), RN1.6 (R6.1)
- net J400 (1): Temp: now also RN1.10 (R7.2), RN1.12 (R5.2), RN1.15 (R2.2); no longer RN1.11 (R6.2), RN1.14 (R3.2)
- net ZD-: now also TP3.1
- net at C3.1, R1.1, U402.6 (-): no longer TP3.1
- net at RN1.8 (R8.1): now also RN1.6 (R6.1); no longer RN1.7 (R7.1)
- net at R418.2, U402.1: now also C1.1
- net at C412.2, R416.1, U402.2 (-): now also C1.2
- net at RN1.13 (R4.2): no longer RN1.15 (R2.2)
- net at RN1.1 (R1.1): now also RN1.3 (R3.1); no longer RN1.2 (R2.1)
- new net: RN1.11 (R6.2), RN1.14 (R3.2)
- no-connect marks 1 -> 2
Other:
- note added: "GND-current compensation 680µA Iq U402"
- note added: "GND-current compensation 762µA RN1"
- note added: "GND-current compensation 9.3mA Iz U401"
- note removed: "GND-current compensation"
- moved on the sheet: C413, D401, R1, R419, U402C

Commit message: Update to REV A
Parts:
- removed JP1: Jumper, Jumper:SolderJumper-2_P1.3mm_Bridged_Pad1.0x1.5mm, symbol Jumper:SolderJumper_2_Bridged
- removed R3: 20R, Resistor_SMD:R_2512_6332Metric, symbol Device:R
- C1: now not fitted
Connections:
- net +7V REF: now also C2.1, U401.3
Other:
- note removed: "Option for LTZ1000 non A"
- note removed: "Option for LTZ1000(A) (open JP1)"
- moved on the sheet: C411, C414

Commit message: Release REV B
Parts:
- added R3, R7: 1k, Resistor_SMD:R_0805_2012Metric, symbol Device:R
- C1: value 10n -> 1n; now fitted
- C2: value 100n -> 10n
- C411: value 22n -> 100n
- C5: value 100n -> 1n; now not fitted
- Q401: Type (none) -> BD139-16
- R1: value 10k -> 1k
- R2: value 680k -> 68k*; Type 30ppm/°C, 300ppm/a LTD - RG -> 10ppm/°C, 100ppm/a LTD - (Susumu URG e.g. URG3216L-683)
- R413: Type 10ppm/°C, 100ppm/a LTD - RG -> 10ppm/°C, 100ppm/a LTD - (Susumu RG3216N-6202)
- R415: value 68k -> 15K*; Type 3ppm/°C, 30ppm/a LTD - URG -> 3ppm/°C, 30ppm/a LTD - VPG VFCP Y163015K (VSMP, FRFC, FRSM,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
- R419: value 1k6 -> 1k43
- R6: value 22k -> 11k8
- RN1: Type TDP1603 -> NOMCT16032001
Connections:
- net +18: now also U402.6 (V+); no longer U402.8 (V+)
- net +7V REF: now also R3.2; no longer Q1.3 (G)
- net GNDA: now also U402.2 (V-); no longer U402.4 (V-)
- net at C411.1, R2.2, R415.2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: now also R7.1; no longer U402.5 (+)
- net at C3.1, R1.1: now also U402.4 (-); no longer U402.6 (-)
- net at C3.2, D400.2 (A): now also U402.5; no longer U402.7
- net at C1.1, R418.2: now also U402.7; no longer U402.1
- net at C1.2, C412.2, R416.1: now also U402.8 (-); no longer U402.2 (-)
- net at R4.1: now also U402.1 (+); no longer U402.3 (+)
- new net: Q1.3 (G), R3.1
- new net: R7.2, U402.3 (+)
Other:
- note added: "GND-current compensation 10.5mA Iz U401"
- note added: "GND-current compensation 680µA Iq U402 490µA Iq Q1 100µA Iq Q2"
- note added: "GND-current compensation 770µA RN1"
- note added: "Simulation shows instability"
- note removed: "GND-current compensation 680µA Iq U402"
- note removed: "GND-current compensation 762µA RN1"
- note removed: "GND-current compensation 9.3mA Iz U401"
- company: (none) -> Michael D.
- title: (none) -> 3458A A9 Reference ADR1000
